File: _autosave-laptop-kicad.kicad_sch (KiCad schematic)
At the start: 25 parts, among them P1 USB_C_Plug, SW1 SW_Push, U1 ATmega32U4-M, Y1 16MHz

Commit message: its 4am dood
Parts:
- removed P1: USB_C_Plug, Connector_USB:USB_C_Plug_JAE_DX07P024AJ1, symbol Connector:USB_C_Plug
- added J1: USB_C_Receptacle_USB2.0, symbol Connector:USB_C_Receptacle_USB2.0
Connections:
- net D+: now also J1.A6 (D+)
- net D-: now also J1.A7 (D-)
- net GND: now also J1.A1 (GND), J1.A12 (GND), J1.B1 (GND), J1.B12 (GND)
- net VCC: now also J1.A4 (VBUS), J1.A9 (VBUS), J1.B4 (VBUS), J1.B9 (VBUS)
- net at R5.1: now also J1.A5 (CC1)
Other:
- moved on the sheet: D1, D2, D3, D4, MX1, MX2, MX3, MX4
