File: laptop-kicad.kicad_pcb (KiCad board)
At the start: 2 copper layers, 42 x 49 mm, 26 parts, among them J1 USB_C_Receptacle_USB2.0, SW1 SW_Push, U1 ATmega32U4-M, Y1 16MHz

Commit message: redoing everything
Parts:
- removed MX3, MX4: MX_SW_HS, PCM_marbastlib-mx:SW_MX_HS_1u
- R6: moved to B.Cu
- moved R6 66.8 mm to (183.2, 64.8), turned to 180 degrees
- moved D3 65.5 mm to (191.4, 47.8)
- moved R5 65.3 mm to (187.3, 64.8)
- moved SW1 60.9 mm to (194.3, 73.5)
- moved D1 58.5 mm to (191.4, 53.7)
- moved D4 51.4 mm to (197.6, 53.9)
- moved R2 51.2 mm to (198.4, 64.8)
- moved R3 51.2 mm to (194.8, 64.8)
- moved C5 49.6 mm to (180.4, 40.3)
- moved C2 49.6 mm to (191.6, 40.3)
- moved D2 46.7 mm to (197.6, 47.8)
- moved C3 36.4 mm to (137.5, 86.4)
- moved C1 28.8 mm to (168.9, 68.3), turned to 90 degrees
- moved C4 27.7 mm to (141.0, 77.2), turned to 90 degrees
- moved C6 23.1 mm to (138.4, 70.7), turned to -90 degrees
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Connections:
- C6 pad 1: GND -> Net-(U1-XTAL1)
- C6 pad 2: Net-(U1-XTAL1) -> GND
- C7 pad 1: GND -> Net-(U1-XTAL2)
- C7 pad 2: Net-(U1-XTAL2) -> GND
- MX2 pad 1: COL0 -> COL1
- R2 pad 1: D+ -> DBUS+
- R3 pad 1: D- -> DBUS-
Routing:
- net +5V: track 0.00 -> 47.8 mm, vias 0 -> 3
- net GND: track 0.00 -> 32.1 mm
- net Net-(U1-~{RESET}): track 0.00 -> 8.02 mm
- net Net-(U1-~{HWB}/PE2): track 0.00 -> 2.94 mm
Other:
- board text added: "Cunny Uohhh ToT"

Commit message: PCB is done pt 2
Parts:
- removed D3, D4: D_Small, Diode_SMD:D_SOD-123
- moved R2 74.3 mm to (124.5, 57.4), turned to -90 degrees
- moved R3 74.0 mm to (121.1, 57.4), turned to -90 degrees
- moved D1 71.3 mm to (121.8, 69.2), turned to 0 degrees
- moved D2 64.4 mm to (136.9, 69.2), turned to 0 degrees
- moved R5 63.5 mm to (125.2, 51.7), turned to -90 degrees
- moved SW1 62.2 mm to (133.5, 86.7)
- moved C2 59.6 mm to (137.3, 64.9), turned to -90 degrees
- moved R6 56.4 mm to (128.4, 51.8), turned to -90 degrees
- moved C5 45.2 mm to (138.0, 55.9), turned to 90 degrees
- moved C1 31.3 mm to (138.7, 59.9), turned to 180 degrees
- moved C4 21.4 mm to (152.6, 59.1)
- moved U1 21.4 mm to (145.3, 61.5)
- moved C3 21.4 mm to (149.1, 68.4)
- moved R1 21.4 mm to (151.3, 65.5)
- moved C6 21.4 mm to (150.2, 52.9)
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Connections:
- C6 pad 1: Net-(U1-XTAL1) -> GND
- C6 pad 2: GND -> Net-(U1-XTAL1)
- C7 pad 1: Net-(U1-XTAL2) -> GND
- C7 pad 2: GND -> Net-(U1-XTAL2)
- U1 pad 38: unconnected-(U1-PF5-Pad38) -> ROW0
- U1 pad 39: unconnected-(U1-PF4-Pad39) -> COL1
- U1 pad 40: unconnected-(U1-PF1-Pad40) -> COL0
Routing:
- net GND: track 32.1 -> 143.9 mm, vias 0 -> 3
- net Net-(U1-~{RESET}): track 8.02 -> 73.3 mm, vias 0 -> 2
- net +5V: track 47.8 -> 94.4 mm, vias 3 -> 6
- net COL0: track 0.00 -> 38.8 mm
- net ROW0: track 0.00 -> 31.9 mm, vias 0 -> 2
- net Net-(U1-D-): track 0.00 -> 23.1 mm
- net Net-(U1-D+): track 0.00 -> 19.5 mm
- net COL1: track 0.00 -> 17.6 mm
- net VBUS: track 0.00 -> 15.8 mm, vias 0 -> 3
- net DBUS-: track 0.00 -> 15.1 mm
- net Net-(D2-A): track 0.00 -> 12.3 mm
- net DBUS+: track 0.00 -> 12.1 mm
- net Net-(D1-A): track 0.00 -> 12.0 mm
- net Net-(U1-XTAL1): track 0.00 -> 8.70 mm
- net Net-(U1-XTAL2): track 0.10 -> 7.99 mm
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Other:
- board text removed: "Cunny Uohhh ToT"

Commit message: Zykrah Edits
Parts:
- moved R2 3.89 mm to (128.4, 57.3)
- moved R3 3.89 mm to (125.0, 57.3)
Routing:
- net Net-(U1-D-): track 23.1 -> 19.3 mm
- net Net-(U1-D+): track 19.5 -> 15.6 mm
- net DBUS-: track 15.1 -> 12.4 mm
- added copper zone on B.Cu, net GND
Changed lines of the file:
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@@
   )
   (footprint "Resistor_SMD:R_0805_2012Metric" (layer "B.Cu")
-    (at 121.125 57.43125 -90)
+    (at 125.014 57.34375 -90)
     (descr "Resistor SMD 0805 (2012 Metric), square (rectangular) end terminal, IPC_7351 nominal, (Body size source: IPC-SM-782 page 72, https://www.pcb-3d.com/wordpress/wp-content/uploads/ipc-sm-782a_amendment_1_and_2.pdf), generated with kicad-footprint-generator")
     (tags "resistor")
@@
   )
   (footprint "Resistor_SMD:R_0805_2012Metric" (layer "B.Cu")
-    (at 124.486 57.40625 -90)
+    (at 128.375 57.31875 -90)
     (descr "Resistor SMD 0805 (2012 Metric), square (rectangular) end terminal, IPC_7351 nominal, (Body size source: IPC-SM-782 page 72, https://www.pcb-3d.com/wordpress/wp-content/uploads/ipc-sm-782a_amendment_1_and_2.pdf), generated with kicad-footprint-generator")
     (tags "resistor")
@@
   (segment (start 149.23125 64.55) (end 151.34375 64.55) (width 0.25) (layer "B.Cu") (net 11))
   (segment (start 141.96875 62.4625) (end 141.383242 62.4625) (width 0.25) (layer "B.Cu") (net 12))
-  (segment (start 130.56875 58.31875) (end 124.486 58.31875) (width 0.25) (layer "B.Cu") (net 12))
+  (segment (start 128.375 58.23125) (end 129.16875 58.23125) (width 0.25) (layer "B.Cu") (net 12))
+  (segment (start 131.21875 60.28125) (end 132.53125 60.28125) (width 0.25) (layer "B.Cu") (net 12))
   (segment (start 138.425 62.325) (end 138.15 62.6) (width 0.25) (layer "B.Cu") (net 12))
   (segment (start 141.383242 62.4625) (end 141.383242 62.491758) (width 0.25) (layer "B.Cu") (net 12))
@@
   (segment (start 138.15 62.6) (end 134.85 62.6) (width 0.25) (layer "B.Cu") (net 12))
   (segment (start 139.630146 62.325) (end 138.425 62.325) (width 0.25) (layer "B.Cu") (net 12))
-  (segment (start 134.85 62.6) (end 130.56875 58.31875) (width 0.25) (layer "B.Cu") (net 12))
+  (segment (start 129.16875 58.23125) (end 131.21875 60.28125) (width 0.25) (layer "B.Cu") (net 12))
+  (segment (start 132.53125 60.28125) (end 134.85 62.6) (width 0.25) (layer "B.Cu") (net 12))
   (segment (start 141.383242 62.491758) (end 139.796904 62.491758) (width 0.25) (layer "B.Cu") (net 12))
-  (segment (start 121.125 58.34375) (end 121.9375 59.15625) (width 0.25) (layer "B.Cu") (net 13))
+  (segment (start 134.726104 63.1125) (end 136.586827 63.1125) (width 0.25) (layer "B.Cu") (net 13))
   (segment (start 136.649327 63.05) (end 138.380945 63.05) (width 0.25) (layer "B.Cu") (net 13))
+  (segment (start 139.44375 62.962195) (end 139.444055 62.9625) (width 0.25) (layer "B.Cu") (net 13))
+  (segment (start 125.014 58.25625) (end 127.489 60.73125) (width 0.25) (layer "B.Cu") (net 13))
+  (segment (start 138.380945 63.05) (end 138.655945 62.775) (width 0.25) (layer "B.Cu") (net 13))
+  (segment (start 132.344854 60.73125) (end 134.726104 63.1125) (width 0.25) (layer "B.Cu") (net 13))
   (segment (start 139.444055 62.9625) (end 141.96875 62.9625) (width 0.25) (layer "B.Cu") (net 13))
-  (segment (start 139.44375 62.962195) (end 139.444055 62.9625) (width 0.25) (layer "B.Cu") (net 13))
-  (segment (start 134.726104 63.1125) (end 136.586827 63.1125) (width 0.25) (layer "B.Cu") (net 13))
-  (segment (start 121.9375 59.15625) (end 130.769854 59.15625) (width 0.25) (layer "B.Cu") (net 13))
   (segment (start 136.586827 63.1125) (end 136.649327 63.05) (width 0.25) (layer "B.Cu") (net 13))
   (segment (start 139.44375 62.775) (end 139.44375 62.962195) (width 0.25) (layer "B.Cu") (net 13))
-  (segment (start 130.769854 59.15625) (end 134.726104 63.1125) (width 0.25) (layer "B.Cu") (net 13))
   (segment (start 138.655945 62.775) (end 139.44375 62.775) (width 0.25) (layer "B.Cu") (net 13))
-  (segment (start 138.380945 63.05) (end 138.655945 62.775) (width 0.25) (layer "B.Cu") (net 13))
+  (segment (start 127.489 60.73125) (end 132.344854 60.73125) (width 0.25) (layer "B.Cu") (net 13))
   (segment (start 131.65625 61.71875) (end 134.15625 59.21875) (width 0.25) (layer "F.Cu") (net 14))
   (segment (start 134.15625 59.21875) (end 135.0625 59.21875) (width 0.25) (layer "F.Cu") (net 14))
@@
   (segment (start 127.3775 48.21625) (end 127.39375 48.2) (width 0.2) (layer "B.Cu") (net 40))
   (segment (start 127.39375 48.2) (end 127.39375 47.34625) (width 0.2) (layer "B.Cu") (net 40))
+  (segment (start 126.84375 48.21625) (end 126.84375 54.875) (width 0.2) (layer "B.Cu") (net 40))
   (segment (start 127.39375 47.34625) (end 127.34375 47.29625) (width 0.2) (layer "B.Cu") (net 40))
-  (segment (start 124.486 56.49375) (end 126.84375 54.136) (width 0.2) (layer "B.Cu") (net 40))
   (segment (start 126.34375 48.16625) (end 126.39375 48.21625) (width 0.2) (layer "B.Cu") (net 40))
-  (segment (start 126.84375 54.136) (end 126.84375 48.21625) (width 0.2) (layer "B.Cu") (net 40))
   (segment (start 126.84375 48.21625) (end 127.3775 48.21625) (width 0.2) (layer "B.Cu") (net 40))
+  (segment (start 126.84375 54.875) (end 128.375 56.40625) (width 0.2) (layer "B.Cu") (net 40))
   (segment (start 125.84375 49.75) (end 126.16375 50.07) (width 0.2) (layer "B.Cu") (net 41))
-  (segment (start 125.84375 47.29625) (end 125.84375 49.75) (width 0.2) (layer "B.Cu") (net 41))
+  (segment (start 126.16375 55.2815) (end 125.014 56.43125) (width 0.2) (layer "B.Cu") (net 41))
+  (segment (start 126.16375 50.07) (end 126.16375 55.2815) (width 0.2) (layer "B.Cu") (net 41))
   (segment (start 126.84375 46.59375) (end 126.84375 47.29625) (width 0.2) (layer "B.Cu") (net 41))
   (segment (start 125.84375 46.42625) (end 125.89375 46.37625) (width 0.2) (layer "B.Cu") (net 41))
-  (segment (start 122.73125 56.51875) (end 121.125 56.51875) (width 0.2) (layer "B.Cu") (net 41))
-  (segment (start 126.16375 50.07) (end 126.16375 53.08625) (width 0.2) (layer "B.Cu") (net 41))
+  (segment (start 125.84375 47.29625) (end 125.84375 49.75) (width 0.2) (layer "B.Cu") (net 41))
   (segment (start 125.84375 47.29625) (end 125.84375 46.42625) (width 0.2) (layer "B.Cu") (net 41))
-  (segment (start 126.16375 53.08625) (end 122.73125 56.51875) (width 0.2) (layer "B.Cu") (net 41))
   (segment (start 125.89375 46.37625) (end 126.62625 46.37625) (width 0.2) (layer "B.Cu") (net 41))
   (segment (start 126.62625 46.37625) (end 126.84375 46.59375) (width 0.2) (layer "B.Cu") (net 41))
   (segment (start 128.34375 47.29625) (end 128.34375 50.8525) (width 0.25) (layer "B.Cu") (net 43))
   (segment (start 128.34375 50.8525) (end 128.35125 50.86) (width 0.25) (layer "B.Cu") (net 43))
+  (zone (net 2) (net_name "GND") (layer "B.Cu") (hatch edge 0.5)
+    (connect_pads (clearance 0.5))
+    (min_thickness 0.25) (filled_areas_thickness no)
+    (fill yes (thermal_gap 0.5) (thermal_bridge_width 0.5))
+    (polygon
+      (pts
+        (xy 113.03 40.64)
+        (xy 156.21 40.64)
+        (xy 156.21 90.17)
+        (xy 113.03 90.17)
+      )
+    )
+  )
 )

Commit message: changing tide
Parts:
- turned C6 to 90 degrees
- turned C7 to -90 degrees
Connections:
- C6 pad 2: Net-(U1-XTAL1) -> GND
Routing:
- net GND: track 143.9 -> 153.3 mm
- net Net-(U1-XTAL2): track 7.99 -> 11.4 mm
Other:
- board text added: "https://osu.ppy.sh/users/18366439"
